File: dac.sch (EAGLE design)
At the start: 68 parts, among them IC1 TLC7733PW, IC2 TC1262-3.3VDB, IC3 LP3879, IC4 XHRA-2HPA, IC5 RCLAMP0502ASMD, IC6 PCM1794, Q1_24 ASF/V_KSC3225KSC, Q2_24M576 ASF/V_KSC3225KSC, Q3_22M5792 ASF/V_KSC3225KSC, U1 OPA1644AIPW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

Commit message: Fix wrong XHRA-2HPA package size
Parts:
- IC4: value XHRA-2HPA -> XHRA-2HPAREAL; device jean:XHRA-2HPA -> jean:XHRA-2HPAREAL
Other:
- moved on the sheet: IC4
Changed lines of the file:
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@@
 <part name="GND1" library="supply1" deviceset="GND" device=""/>
 <part name="PE1" library="supply1" deviceset="PE" device=""/>
-<part name="IC4" library="jean" deviceset="XHRA-2HPA" device=""/>
+<part name="IC4" library="jean" deviceset="XHRA-2HPA" device="REAL" value="XHRA-2HPAREAL"/>
 <part name="GND2" library="supply1" deviceset="GND" device=""/>
 <part name="GND3" library="supply1" deviceset="GND" device=""/>
